File: Kicad_Project/ContollerBoard2/ControllerBoard2.kicad_pcb (KiCad board)
At the start: 2 copper layers, 26.2 x 43.2 mm, 35 parts, among them J1 Main Header, J2 SWD, J3 WD_Disable, Q1 BSS84, U1 FS32K116, U2 UJA1075A

Commit message: First draft of controlboard2
Parts:
- removed C5: 100n, Capacitor_SMD:C_0603_1608Metric_Pad1.05x0.95mm_HandSolder
- removed C8: 4.7n, Capacitor_SMD:C_0805_2012Metric_Pad1.15x1.40mm_HandSolder
- removed R3, R4: 1.3k, Resistor_SMD:R_0603_1608Metric_Pad1.05x0.95mm_HandSolder
- added C2: 18p, Capacitor_SMD:C_0603_1608Metric_Pad1.05x0.95mm_HandSolder, F.Cu at (123.6, 105.3)
- added C3: 18p, Capacitor_SMD:C_0603_1608Metric_Pad1.05x0.95mm_HandSolder, F.Cu at (123.6, 94.1)
- added Y1: 8Mhz, Crystal:Crystal_SMD_Abracon_ABM3-2Pin_5.0x3.2mm_HandSoldering, F.Cu at (123.6, 99.6)
- U1: value FS32K116 -> STM32F303K8Tx; footprint digikey-footprints:LQFP-48_7x7mm -> Package_QFP:LQFP-32_7x7mm_P0.8mm
- U2: value UJA1075A -> UJA1075A-3.3
- moved C4 3.37 mm to (127.1, 91.8), turned to 0 degrees
- moved C1 3.29 mm to (137.7, 101.8), turned to 90 degrees
- moved U1 2.31 mm to (131.7, 98.0), turned to 180 degrees
- moved U2 0.10 mm to (132.0, 85.3)
Connections:
- C1 pad 2: +5V -> +3V3
- C4 pad 1: +5V -> +3V3
- C6 pad 1: +5V -> +3V3
- D1 pad 2: +5V -> +3V3
- D2 pad 2: PTA13 -> (no net)
- D3 pad 2: PTA12 -> (no net)
- D5 pad 2: +5V -> +3V3
- J1 pad 10: PTA2 -> (no net)
- J1 pad 11: PTA7 -> (no net)
- J1 pad 12: I2C_SDA -> (no net)
- J1 pad 13: I2C_SCL -> (no net)
- J1 pad 14: PTA1 -> (no net)
- J1 pad 15: PTA0 -> (no net)
- J1 pad 16: PTA11 -> (no net)
- J1 pad 20: +5V -> (no net)
- J1 pad 21: PTC14 -> (no net)
- J1 pad 22: PTC15 -> PA3
- J1 pad 23: PTC16 -> PA2
- J1 pad 24: PTC1 -> PA1
- J1 pad 25: PTC2 -> PA0
- J1 pad 26: PTC3 -> (no net)
- J1 pad 27: PTB4 -> (no net)
- J1 pad 28: PTB5 -> PB7
- J1 pad 29: PTD16 -> PB6
- J1 pad 30: PTD0 -> PB5
- J1 pad 31: PTD1 -> PB4
- J1 pad 6: PTB13 -> (no net)
- J1 pad 7: PTD3 -> (no net)
- J1 pad 8: PTD2 -> (no net)
- J1 pad 9: PTA3 -> (no net)
- J2 pad 1: +5V -> +3V3
- J3 pad 2: +5V -> +3V3
- Q1 pad 2: +5V -> +3V3
- R1 pad 1: +5V -> +3V3
- R13 pad 1: +5V -> +3V3
- R5 pad 1: +5V -> +3V3
- R6 pad 1: +5V -> +3V3
- R7 pad 1: +5V -> +3V3
- U1 pad 1: PTD1 -> +3V3
- U1 pad 10: PTD16 -> SCSN
- U1 pad 11: (no net) -> SCK
- U1 pad 12: (no net) -> MISO
- U1 pad 13: (no net) -> MOSI
- U1 pad 14: PTB5 -> (no net)
- U1 pad 15: PTB4 -> (no net)
- U1 pad 16: PTC3 -> GND
- U1 pad 17: PTC2 -> +3V3
- U1 pad 18: SBC_INTN -> (no net)
- U1 pad 19: PTC1 -> (no net)
- U1 pad 2: PTD0 -> OSC_IN
- U1 pad 20: PTC16 -> (no net)
- U1 pad 21: PTC15 -> CAN_RX
- U1 pad 22: PTC14 -> CAN_TX
- U1 pad 23: MISO -> SWDIO
- U1 pad 24: SCK -> SWDCLK
- U1 pad 25: MOSI -> TDI
- U1 pad 26: SCSN -> SWO
- U1 pad 27: (no net) -> PB4
- U1 pad 28: (no net) -> PB5
- U1 pad 29: PTA7 -> PB6
- U1 pad 3: CAN_TX -> OSC_OUT
- U1 pad 30: GND -> PB7
- U1 pad 31: +5V -> (no net)
- U1 pad 32: PTB13 -> GND
- U1 pad 4: CAN_RX -> RESET
- U1 pad 5: +5V -> +3V3
- U1 pad 6: +5V -> PA0
- U1 pad 7: GND -> PA1
- U1 pad 8: I2C_SCL -> PA2
- U1 pad 9: I2C_SDA -> PA3
- U2 pad 24: SPLIT -> (no net)
- U2 pad 29: +5V -> +3V3
- U2 pad 4: +5V -> +3V3
- U2 pad 7: SBC_INTN -> (no net)
Routing:
- net +5V: track 101.6 -> 0.00 mm, vias 5 -> 0
- net +3V3: track 0.00 -> 93.4 mm, vias 0 -> 4
- net I2C_SCL: track 19.3 -> 0.00 mm
- net I2C_SDA: track 18.9 -> 0.00 mm
- net PTA11: track 18.4 -> 0.00 mm
- net PB4: track 0.00 -> 17.3 mm
- net GND: track 19.3 -> 2.21 mm, vias 22 -> 9
- net OSC_IN: track 0.00 -> 17.0 mm, vias 0 -> 2
- net OSC_OUT: track 0.00 -> 16.8 mm, vias 0 -> 2
- net PTA7: track 16.7 -> 0.00 mm, vias 2 -> 0
- net PTC14: track 14.7 -> 0.00 mm
- net SBC_INTN: track 14.6 -> 0.00 mm, vias 2 -> 0
- net PB5: track 0.00 -> 14.5 mm
- net PTD1: track 13.4 -> 0.00 mm
- net PTA0: track 13.3 -> 0.00 mm
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Other:
- board text added: "UBCO MOTORSPORTS CONTROLBOARD V2"
- board text removed: "UBCO MOTORSPORTS CONTROLBOARD V1.1"
